File: 1512hh-control.kicad_pcb (KiCad board)
At the start: 2 copper layers, 0 parts

Commit message: Route and layout board
Parts:
- added BZ1: Buzzer, A_Project_Library:PKM22EPPH4, F.Cu at (63.5, 73.4)
- added C1: 10uF 0603, Capacitor_SMD:C_0603_1608Metric, F.Cu at (73.5, 85.5)
- added C2: 0.1uF 0603, Capacitor_SMD:C_0603_1608Metric, F.Cu at (22.5, 95.0)
- added C3: 1uF 0603, Capacitor_SMD:C_0603_1608Metric, F.Cu at (29.5, 100.6)
- added C4: 220uF 6.3V, Capacitor_THT:C_Radial_D6.3mm_H11.0mm_P2.50mm, F.Cu at (116.0, 111.0)
- added C5: 22uF 6.3V, Capacitor_THT:C_Radial_D5.0mm_H11.0mm_P2.00mm, F.Cu at (93.0, 113.5)
- added C6: 10uF 6.3V, Capacitor_THT:C_Radial_D5.0mm_H11.0mm_P2.00mm, F.Cu at (25.5, 102.5)
- added C7: 220uF 6.3V, Capacitor_THT:C_Radial_D6.3mm_H11.0mm_P2.50mm, F.Cu at (126.5, 111.0)
- added D1: LED, LED_THT:LED_D3.0mm, F.Cu at (93.8, 82.3)
- added D10: LED, LED_THT:LED_D3.0mm, F.Cu at (185.0, 82.5)
- added D11: LED, LED_THT:LED_D3.0mm, F.Cu at (193.5, 82.5)
- added D12: LED, LED_THT:LED_D3.0mm, F.Cu at (213.5, 82.2)
- added D13: LED, LED_THT:LED_D3.0mm, F.Cu at (230.5, 82.5)
- added D14: D_Zener_Dual_CommonAnode_KKA, Package_TO_SOT_SMD:SOT-23, F.Cu at (75.5, 65.9)
- added D15: LED_RGKB, LED_THT:LED_D5.0mm-4_RGB, F.Cu at (259.0, 97.7)
- added D2: LED, LED_THT:LED_D3.0mm, F.Cu at (102.5, 82.3)
- added D3: LED, LED_THT:LED_D3.0mm, F.Cu at (111.0, 82.2)
- added D4: LED, LED_THT:LED_D3.0mm, F.Cu at (119.5, 82.3)
- added D5: LED, LED_THT:LED_D3.0mm, F.Cu at (128.0, 82.2)
- added D6: LED, LED_THT:LED_D3.0mm, F.Cu at (139.5, 82.2)
- added D7: LED, LED_THT:LED_D3.0mm, F.Cu at (148.0, 82.3)
- added D8: LED, LED_THT:LED_D3.0mm, F.Cu at (156.5, 82.5)
- added D9: LED, LED_THT:LED_D3.0mm, F.Cu at (176.5, 82.5)
- added G***: LOGO, LOGO, F.Cu at (52.2, 89.3)
- added G***: LOGO, LOGO, F.Cu at (254.8, 81.5)
- added J1: Conn_02x03_Odd_Even, Connector_PinHeader_2.54mm:PinHeader_2x03_P2.54mm_Vertical, F.Cu at (24.0, 67.5)
- added J2: Conn_01x05_Male, Connector_JST:JST_XH_S5B-XH-A-1_1x05_P2.50mm_Horizontal, F.Cu at (253.5, 108.0)
- added J3: Conn_01x06_Male, Connector_JST:JST_XH_S6B-XH-A-1_1x06_P2.50mm_Horizontal, F.Cu at (33.5, 109.4)
- added J4: Conn_01x02_Male, Connector_JST:JST_XH_S2B-XH-A-1_1x02_P2.50mm_Horizontal, F.Cu at (143.2, 108.2)
- added Q1: BSS84, Package_TO_SOT_SMD:SOT-23, F.Cu at (53.5, 115.4)
- added Q2: BSS84, Package_TO_SOT_SMD:SOT-23, F.Cu at (26.4, 115.5)
- added Q3: 2N7002, Package_TO_SOT_SMD:SOT-23, F.Cu at (53.5, 109.9)
- added Q4: 2N7002, Package_TO_SOT_SMD:SOT-23, F.Cu at (26.4, 110.5)
- added R1: 500 0603, Resistor_SMD:R_0603_1608Metric, F.Cu at (93.0, 76.5)
- added R10: 500 0603, Resistor_SMD:R_0603_1608Metric, F.Cu at (184.2, 76.5)
- added R11: 500 0603, Resistor_SMD:R_0603_1608Metric, F.Cu at (192.7, 76.5)
- added R12: 300 0603, Resistor_SMD:R_0603_1608Metric, F.Cu at (212.5, 76.8)
- added R13: 300 0603, Resistor_SMD:R_0603_1608Metric, F.Cu at (229.5, 77.0)
- added R14: 3K 0603, Resistor_SMD:R_0603_1608Metric, F.Cu at (245.5, 113.5)
- added R15: 3K 0603, Resistor_SMD:R_0603_1608Metric, F.Cu at (245.5, 109.5)
- added R16: 4.7K 0603, Resistor_SMD:R_0603_1608Metric, F.Cu at (245.5, 105.5)
- added R17: 4.7K 0603, Resistor_SMD:R_0603_1608Metric, F.Cu at (134.2, 110.6)
- added R18: 10K 0603, Resistor_SMD:R_0603_1608Metric, F.Cu at (26.9, 97.9)
- added R19: 3K 0603, Resistor_SMD:R_0603_1608Metric, F.Cu at (131.8, 106.3)
- added R2: 300 0603, Resistor_SMD:R_0603_1608Metric, F.Cu at (101.7, 76.5)
- added R20: 3K 0603, Resistor_SMD:R_0603_1608Metric, F.Cu at (134.9, 106.3)
- added R21: 4.7K 0603, Resistor_SMD:R_0603_1608Metric, F.Cu at (138.0, 106.2)
- added R22: 0 0603, Resistor_SMD:R_0603_1608Metric, F.Cu at (50.0, 76.5)
- added R23: 132 0603, Resistor_SMD:R_0603_1608Metric, F.Cu at (249.4, 90.5)
- added R24: 132 0603, Resistor_SMD:R_0603_1608Metric, F.Cu at (249.5, 94.0)
- added R25: 132 0603, Resistor_SMD:R_0603_1608Metric, F.Cu at (249.5, 97.5)
- added R26: 10K 0603, Resistor_SMD:R_0603_1608Metric, F.Cu at (57.4, 112.0)
- added R27: 10K 0603, Resistor_SMD:R_0603_1608Metric, F.Cu at (23.0, 111.0)
- added R28: 10K 0603, Resistor_SMD:R_0603_1608Metric, F.Cu at (37.5, 103.0)
- added R29: 3K 0603, Resistor_SMD:R_0603_1608Metric, F.Cu at (37.5, 99.8)
- added R3: 300 0603, Resistor_SMD:R_0603_1608Metric, F.Cu at (110.2, 76.5)
- added R30: 4.7K 0603, Resistor_SMD:R_0603_1608Metric, F.Cu at (34.1, 100.6)
- added R4: 300 0603, Resistor_SMD:R_0603_1608Metric, F.Cu at (118.7, 76.5)
- added R5: 500 0603, Resistor_SMD:R_0603_1608Metric, F.Cu at (127.2, 76.5)
- added R6: 500 0603, Resistor_SMD:R_0603_1608Metric, F.Cu at (138.8, 76.8)
- added R7: 500 0603, Resistor_SMD:R_0603_1608Metric, F.Cu at (147.2, 76.8)
- added R8: 500 0603, Resistor_SMD:R_0603_1608Metric, F.Cu at (155.8, 76.8)
- added R9: 500 0603, Resistor_SMD:R_0603_1608Metric, F.Cu at (175.8, 76.5)
- added SW1: SW_Push, Button_Switch_THT:SW_PUSH_6mm_H5mm, F.Cu at (70.5, 93.2)
- added SW2: SW_Push, Button_Switch_THT:SW_PUSH_6mm_H5mm, F.Cu at (107.5, 93.5)
- added SW3: SW_Push, Button_Switch_THT:SW_PUSH_6mm_H5mm, F.Cu at (144.7, 93.3)
- added SW4: SW_Push, Button_Switch_THT:SW_PUSH_6mm_H5mm, F.Cu at (181.8, 93.2)
- added SW5: SW_Push, Button_Switch_THT:SW_PUSH_6mm_H5mm, F.Cu at (218.8, 93.2)
- added U1: NPIC6C596ADJ, Package_SO:SOIC-16_3.9x9.9mm_P1.27mm, F.Cu at (82.1, 83.0)
- added U2: AMS1117-3.3, Package_TO_SOT_SMD:SOT-223-3_TabPin2, F.Cu at (105.0, 112.0)
- added U3: ESP32-WROOM-32, RF_Module:ESP32-WROOM-32, F.Cu at (29.5, 81.5)
Routing:
- net /P5V: track 0.00 -> 600.4 mm, vias 0 -> 8
- net /DUST_3V3_OUT: track 0.00 -> 321.5 mm, vias 0 -> 2
- net /LED_HEPA: track 0.00 -> 232.6 mm
- net /LED_G: track 0.00 -> 230.7 mm
- net /LED_B: track 0.00 -> 228.9 mm
- net /LED_R: track 0.00 -> 228.0 mm
- net /LED_ODOR: track 0.00 -> 227.2 mm
- net /SW_FILTER: track 0.00 -> 199.0 mm
- net /SW_TIMER: track 0.00 -> 158.7 mm
- net Net-(D11-Pad1): track 0.00 -> 130.9 mm
- net /DOOR_3V3_OUT: track 0.00 -> 127.4 mm
- net Net-(D10-Pad1): track 0.00 -> 120.3 mm
- net /SW_ION: track 0.00 -> 119.5 mm
- net Net-(D9-Pad1): track 0.00 -> 109.0 mm
- net /P3V3: track 0.00 -> 107.2 mm
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- added copper zone on F.Cu, net /P3V3
- added copper zone on B.Cu, net GND
- added copper zone on F.Cu, net GND
Other:
- board outline added: 259.5 x 60.7 mm
- board text added: "(5V PWM)"
- board text added: "1h"
- board text added: "4h"
- board text added: "5V"
- board text added: "5V SW"
- board text added: "8h"
- board text added: "Auto"
- board text added: "D2,D3,D4,RGB,HEPA/Odor: Direct Other: SR"
- board text added: "Door Sw"
- board text added: "Dust Sensor"
- board text added: "Eco"
- board text added: "FG"
- board text added: "GND"
- board text added: "HEPA"
- board text added: "ION"
- board text added: "ION, M_EN 5V Active H FG 5V SqWave PWM 2.5-3.3V 25-85%"
- board text added: "Ion"
- board text added: "M_EN"
- board text added: "NC"
- board text added: "NPIC6C596 SOIC 16"
- board text added: "OUT"
- board text added: "Odor"
- board text added: "PWM"
- board text added: "Power"
- board text added: "Power PCB"
- board text added: "Prog"
- board text added: "RGB LED (IAQ)"
- board text added: "Reset"
- board text added: "S1"
- board text added: "S2"
- board text added: "S3"
- board text added: "Speed"
- board text added: "Timer"
