File: 1512hh-control.kicad_sch (KiCad schematic)
At the start: 64 parts, among them J1 Conn_01x06_Male, J2 Conn_02x03_Odd_Even, J3 Conn_01x05_Male, J4 Conn_01x02_Male, Q1 2N7002, Q2 BSS84, Q3 2N7002, Q4 BSS84, SW1 SW_Push, SW2 SW_Push, SW3 SW_Push, SW4 SW_Push, SW5 SW_Push, SW6 SW_Push, U1 AMS1117-3.3, U2 ESP32-WROOM-32, U3 NPIC6C596ADJ

Commit message: Route and layout board
Parts:
- added D12, D13: LED, LED_THT:LED_D3.0mm, symbol Device:LED
- added D14: D_Zener_Dual_CommonAnode_KKA, Package_TO_SOT_SMD:SOT-23, symbol Device:D_Zener_Dual_CommonAnode_KKA
- added R12, R13: 300 0603, Resistor_SMD:R_0603_1608Metric, symbol Device:R
- added R22: 0 0603, Resistor_SMD:R_0603_1608Metric, symbol Device:R
- BZ1: footprint (none) -> A_Project_Library:PKM22EPPH4
- C3: renamed from C5; footprint Capacitor_THT:C_Radial_D6.3mm_H11.0mm_P2.50mm -> Capacitor_SMD:C_0603_1608Metric
- renumbered C7 to C1, C6 to C2, C1 to C4, C3 to C5, C4 to C6, C2 to C7, D9 to D11, D8 to D15, D5 to D2, D6 to D3, D7 to D4, D2 to D5, D3 to D6, D4 to D7, D12 to D8, D11 to D9, J2 to J1, J3 to J2, J1 to J3, Q2 to Q1, Q4 to Q2, Q1 to Q3, Q3 to Q4, R10 to R1, R25 to R10, R24 to R11, R4 to R14, R6 to R15, R5 to R16, R22 to R17, R2 to R18, R20 to R19, R14 to R2, R23 to R20, R17 to R23, R18 to R24, R19 to R25, R1 to R26, R3 to R27, R7 to R28, R8 to R29, R15 to R3, R9 to R30, R16 to R4, R11 to R5, R12 to R6, R13 to R7, R27 to R8, R26 to R9, SW2 to SW1, SW3 to SW2, SW4 to SW3, SW5 to SW4, SW6 to SW5, SW1 to SW6, U3 to U1, U1 to U2, U2 to U3
Connections:
- net 15VEN_3V3_IN: now also U3.7 (IO35); no longer U3.30 (IO18)
- net DOOR_3V3_OUT: now also U3.8 (IO32); no longer U3.9 (IO33)
- net DUST_3V3_OUT: now also U3.31 (IO19); no longer U3.24 (IO2)
- net FAN_FG_3V: now also U3.5 (SENSOR_VN); no longer U3.36 (IO22)
- net FAN_PWM_3V3_OUT: now also U3.6 (IO34); no longer U3.33 (IO21)
- net GND: now also D12.1 (K), D13.1 (K)
- net ION_3V3_IN: now also U3.4 (SENSOR_VP); no longer U3.37 (IO23)
- net LED_B: now also U3.13 (IO14); no longer U3.8 (IO32)
- net LED_G: now also U3.9 (IO33); no longer U3.7 (IO35)
- net LED_H: now also U3.22 (SDI/SD1); no longer U3.12 (IO27)
- net LED_L: now also U3.24 (IO2); no longer U3.17 (SHD/SD2)
- net LED_M: now also U3.23 (IO15); no longer U3.18 (SWP/SD3)
- net LED_R: now also U3.12 (IO27); no longer U3.6 (IO34)
- net SHIFT_DAT_ESP2SR: now also U3.26 (IO4); no longer U3.27 (IO16)
- net SHIFT_MR_ESP2SR: now also U3.27 (IO16); no longer U3.26 (IO4)
- net SW_FILTER: now also U3.17 (SHD/SD2); no longer U3.19 (SCS/CMD)
- net SW_ION: now also U3.19 (SCS/CMD); no longer U3.21 (SDO/SD0)
- net SW_POWER: now also U3.21 (SDO/SD0); no longer U3.23 (IO15)
- net SW_SPEED: now also U3.20 (SCK/CLK); no longer U3.22 (SDI/SD1)
- net SW_TIMER: now also U3.18 (SWP/SD3); no longer U3.20 (SCK/CLK)
- net at BZ1.1 (-): now also D14.2 (K), R22.2; no longer U3.10 (IO25)
- net at BZ1.2 (+), U3.11 (IO26): now also D14.1 (K)
- net LED_ODOR: now reaches U3.14 (IO12)
- net LED_ODOR: now also R13.1
- net LED_HEPA: now reaches U3.16 (IO13)
- net LED_HEPA: now also R12.1
- new net: D13.2 (A), R13.2
- new net: R22.1, U3.10 (IO25)
- new net: D12.2 (A), R12.2
- no-connect marks 7 -> 3
Other:
- moved on the sheet: BZ1, SW1, SW2, SW3, SW4, SW5
